File: hardware/SmartBeehive.kicad_sch (KiCad schematic)
At the start: 7 parts, among them U1 ESP32-S3-DevKitC, U2 HX711_Module, U3 SSD1306, U4 DS18B20, U5 INMP441, U6 SHT31

Commit message: Add SmartBeehiveLib footprints for HX711 and SSD1306, and update library references
Parts:
- U2: footprint (none) -> SmartBeehiveLib:HX711
- U3: footprint (none) -> SmartBeehiveLib:SSD1306
Changed lines of the file:
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@@
 			)
 		)
-		(property "Footprint" ""
+		(property "Footprint" "SmartBeehiveLib:SSD1306"
 			(at 231.14 144.78 0)
 			(hide yes)
@@
 			)
 		)
-		(property "Footprint" ""
+		(property "Footprint" "SmartBeehiveLib:HX711"
 			(at 201.93 68.58 0)
 			(hide yes)

Commit message: Add HX711_V2 footprint and update SSD1306 UUIDs; fix SmartBeehive schematic and lock file
Parts:
- U2: footprint SmartBeehiveLib:HX711 -> SmartBeehiveLib:HX711_V2
Connections:
- no-connect marks 30 -> 36
Changed lines of the file:
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@@
+	)
+	(no_connect
+		(at 210.82 72.39)
 	)
 	(no_connect
@@
 	)
 	(no_connect
+		(at 210.82 74.93)
+	)
+	(no_connect
 		(at 161.29 72.39)
 	)
@@
 	)
 	(no_connect
+		(at 210.82 69.85)
+	)
+	(no_connect
 		(at 161.29 82.55)
 	)
@@
 	)
 	(no_connect
+		(at 210.82 64.77)
+	)
+	(no_connect
 		(at 161.29 110.49)
 	)
@@
 	)
 	(no_connect
+		(at 210.82 67.31)
+	)
+	(no_connect
 		(at 161.29 95.25)
 	)
@@
 	(no_connect
 		(at 161.29 46.99)
+	)
+	(no_connect
+		(at 210.82 62.23)
 	)
 	(no_connect
@@
 	)
 	(symbol
-		(lib_id "HX711_BreakOut:HX711_BreakOut_1")
-		(at 201.93 68.58 0)
-		(unit 1)
-		(body_style 1)
-		(exclude_from_sim no)
-		(in_bom yes)
-		(on_board yes)
-		(in_pos_files yes)
-		(dnp no)
-		(fields_autoplaced yes)
-		(property "Reference" "U2"
-			(at 209.55 67.3099 0)
-			(show_name no)
-			(do_not_autoplace no)
-			(effects
-				(font
-					(size 1.27 1.27)
-				)
-				(justify left)
-			)
-		)
-		(property "Value" "HX711_Module"
-			(at 209.55 69.8499 0)
-			(show_name no)
-			(do_not_autoplace no)
-			(effects
-				(font
-					(size 1.27 1.27)
-				)
-				(justify left)
-			)
-		)
-		(property "Footprint" "SmartBeehiveLib:HX711"
-			(at 201.93 68.58 0)
-			(hide yes)
-			(show_name no)
-			(do_not_autoplace no)
-			(effects
-				(font
-					(size 1.27 1.27)
-				)
-			)
-		)
-		(property "Datasheet" ""
-			(at 201.93 68.58 0)
-			(hide yes)
-			(show_name no)
-			(do_not_autoplace no)
-			(effects
-				(font
-					(size 1.27 1.27)
-				)
-			)
-		)
-		(property "Description" ""
-			(at 201.93 68.58 0)
-			(hide yes)
-			(show_name no)
-			(do_not_autoplace no)
-			(effects
-				(font
-					(size 1.27 1.27)
-				)
-			)
-		)
-		(pin "3"
-		)
-		(pin "2"
-		)
-		(pin "1"
-		)
-		(pin "4"
-		)
-		(instances
-			(project "SmartBeehive"
-				(path "/d27290ed-e962-41b2-a92d-f7a6144dd72d"
-					(reference "U2")
-					(unit 1)
-				)
-			)
-		)
-	)
-	(symbol
 		(lib_id "power:GND")
 		(at 135.89 135.89 0)
@@
 					(unit 1)
 				)
+			)
+		)
+	)
+	(symbol
+		(lib_id "HX711_BreakOut:HX711_BreakOut_1")
+		(at 201.93 68.58 0)
+		(unit 1)
+		(body_style 1)
+		(exclude_from_sim no)
+		(in_bom yes)
+		(on_board yes)
+		(in_pos_files yes)
+		(dnp no)
+		(fields_autoplaced yes)
+		(property "Reference" "U2"
+			(at 204.0733 55.88 0)
+			(show_name no)
+			(do_not_autoplace no)
+			(effects
+				(font
+					(size 1.27 1.27)
+				)
+				(justify left)
+			)
+		)
+		(property "Value" "HX711_Module"
+			(at 204.0733 58.42 0)
+			(show_name no)
+			(do_not_autoplace no)
+			(effects
+				(font
+					(size 1.27 1.27)
+				)
+				(justify left)
+			)
+		)
+		(property "Footprint" "SmartBeehiveLib:HX711_V2"
+			(at 201.93 68.58 0)
+			(hide yes)
+			(show_name no)
+			(do_not_autoplace no)
+			(effects
+				(font
+					(size 1.27 1.27)
+				)
+			)
+		)
+		(property "Datasheet" ""
+			(at 201.93 68.58 0)
+			(hide yes)
+			(show_name no)
+			(do_not_autoplace no)
+			(effects
+				(font
+					(size 1.27 1.27)
+				)
+			)
+		)
+		(property "Description" ""
+			(at 201.93 68.58 0)
+			(hide yes)
+			(show_name no)
+			(do_not_autoplace no)
+			(effects
+				(font
+					(size 1.27 1.27)
+				)
+			)
+		)
+		(pin "7"
+		)
+		(pin "2"
+		)
+		(pin "5"
+		)
+		(pin "6"
+		)
+		(pin "1"
+		)
+		(pin "4"
+		)
+		(pin "3"
+		)
+		(pin "8"
+		)
+		(pin "9"
+		)
+		(pin "10"
+		)
+		(instances
+			(project "SmartBeehive"
+				(path "/d27290ed-e962-41b2-a92d-f7a6144dd72d"
+					(reference "U2")
+					(unit 1)
+				)

Commit message: Refactor SHT31 symbol pin assignments and add footprint to SmartBeehiveLib
Parts:
- U6: footprint (none) -> SmartBeehiveLib:SHT31
Connections:
- net +3V3: now also U6.4 (VIN); no longer U6.1 (VIN)
- net GND: now also U6.3 (GND); no longer U6.2 (GND)
- net at U1.27 (GPIO21), U3.3 (SCL): now also U6.2 (SCL); no longer U6.3 (SCL)
- net at U1.35 (GPIO38), U3.4 (SDA): now also U6.1 (SDA); no longer U6.4 (SDA)
Changed lines of the file:
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@@
 			)
 		)
-		(property "Footprint" ""
+		(property "Footprint" "SmartBeehiveLib:SHT31"
 			(at 201.93 144.78 0)
 			(hide yes)

Commit message: Add footprints for INMP441 and DS18B20; update schematic properties
Parts:
- U4: footprint (none) -> SmartBeehiveLib:DS18B20
- U5: footprint (none) -> SmartBeehiveLib:INMP441
Changed lines of the file:
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@@
 			)
 		)
-		(property "Footprint" ""
+		(property "Footprint" "SmartBeehiveLib:INMP441"
 			(at 66.04 63.5 0)
 			(hide yes)
@@
 			)
 		)
-		(property "Footprint" ""
+		(property "Footprint" "SmartBeehiveLib:DS18B20"
 			(at 231.14 100.33 0)
 			(hide yes)
